Commit message: update
nav2d/registration combined with direct UI command
nav2d/lift_client added
Arduino code backup
modified sick_tim code backup

File: sick_tim/urdf/sick_tim.urdf.xacro (robot description, xacro)
@@ -4,17 +4,19 @@
   xmlns:sensor="http://playerstage.sourceforge.net/gazebo/xmlschema/#sensor"
   xmlns:xacro="http://ros.org/wiki/xacro">
-  <xacro:macro name="sick_tim310" params="name ros_topic">
+  <xacro:macro name="sick_tim310" params="name ros_topic min_angle:=-2.357 max_angle:=2.357 min_range:=0.05 max_range:=4.0">
     <xacro:sick_tim name="${name}" ros_topic="${ros_topic}"
       length="0.06" width="0.06" height="0.079" mass="0.150" z_offset="0.05595"
-      min_range="0.05" max_range="4.0"
+      min_angle="${min_angle}" max_angle="${max_angle}"
+      min_range="${min_range}" max_range="${max_range}"
       mesh="package://sick_tim/meshes/sick_tim310.stl" />
   </xacro:macro>
-  <xacro:macro name="sick_tim551" params="name ros_topic">
+  <xacro:macro name="sick_tim551" params="name ros_topic min_angle:=-2.357 max_angle:=2.357 min_range:=0.05 max_range:=10">
     <xacro:sick_tim name="${name}" ros_topic="${ros_topic}"
       length="0.06" width="0.06" height="0.086" mass="0.250" z_offset="0.06296"
-      min_range="0.05" max_range="10.0"
+      min_range="${min_range}" max_range="${max_range}"
+      min_angle="${min_angle}" max_angle="${max_angle}"
       mesh="package://sick_tim/meshes/sick_tim551.stl" />
   </xacro:macro>
-  <xacro:macro name="sick_tim" params="name ros_topic length width height mass z_offset min_range max_range mesh">
+  <xacro:macro name="sick_tim" params="name ros_topic length width height mass z_offset min_angle max_angle min_range max_range mesh">
     <!-- z_offset: distance between base plate and laser center (= center of mesh) -->
     <link name="${name}_mount_link">
@@ -53,5 +55,5 @@
       </inertial>
     </link>
-    <xacro:sick_tim_laser_gazebo_v0 name="${name}" link="${name}" ros_topic="${ros_topic}" update_rate="15.0" min_angle="-2.357" max_angle="2.357" min_range="${min_range}" max_range="${max_range}"/>
+    <xacro:sick_tim_laser_gazebo_v0 name="${name}" link="${name}" ros_topic="${ros_topic}" update_rate="15.0" min_angle="${min_angle}" max_angle="${max_angle}" min_range="${min_range}" max_range="${max_range}"/>
   </xacro:macro>
   <xacro:macro name="sick_tim_laser_gazebo_v0" params="name link ros_topic update_rate min_angle max_angle min_range max_range">
