Commit message: update

File: navigation_2d/nav2d_run/param/UAGV.urdf.xacro (robot description, xacro)
@@ -26,4 +26,4 @@
   <xacro:include filename="$(find sick_tim)/urdf/sick_tim.urdf.xacro" />
   <!--xacro:sick_tim310 name="base_laser_link" ros_topic="scan" /-->
-  <xacro:sick_tim name="laser" ros_topic="scan" length="0.06" width="0.06" height="0.086" mass="0.250" z_offset="0.06296" min_range="0.05" max_range="10.0" mesh="file://$(find sick_tim)/meshes/sick_tim551.stl"/>
+  <xacro:sick_tim name="laser" ros_topic="scan" length="0.06" width="0.06" height="0.086" mass="0.250" z_offset="0.06296" min_angle="-2.357" max_angle="2.357" min_range="0.05" max_range="10.0" mesh="file://$(find sick_tim)/meshes/sick_tim551.stl"/>
 </robot>

File: sick_tim/urdf/sick_tim.urdf.xacro (robot description, xacro)
@@ -20,5 +20,5 @@
   <xacro:macro name="sick_tim" params="name ros_topic length width height mass z_offset min_angle max_angle min_range max_range mesh">
     <!-- z_offset: distance between base plate and laser center (= center of mesh) -->
-    <link name="${name}_mount_link">
+    <link name="${name}_link">
       <inertial>
         <mass value="0.001" />
@@ -29,5 +29,5 @@
     </link>
     <joint name="${name}_joint" type="fixed">
-      <parent link="${name}_mount_link" />
+      <parent link="${name}_link" />
       <child link="${name}" />
       <origin rpy="0 0 0" xyz="0 0 ${z_offset}"/>
